File: hardware/kicad/obsonet-wireless/obsonet-wireless.kicad_sch (KiCad schematic)
At the start: 22 parts, among them U1 EP1C3T100C8N, U2 AM29F010B

Commit message: wiring EPCS to config the FPGA
Parts:
- added C11: 100nF, Capacitor_SMD:C_0805_2012Metric_Pad1.18x1.45mm_HandSolder, symbol Device:C
- added C13, C14, C15, C16, C17: 0.1uF, Capacitor_SMD:C_0805_2012Metric, symbol Device:C
- added J1: Conn_02x05_Odd_Even, Connector_PinHeader_2.54mm:PinHeader_2x05_P2.54mm_Vertical, symbol Connector_Generic:Conn_02x05_Odd_Even
- added R1: 10, Resistor_SMD:R_0805_2012Metric, symbol Device:R
- added RN9: 10K, Resistor_SMD:R_Array_Convex_4x0603, symbol Device:R_Pack04_Split
- added U3: EPCS1SI8N, libraries:SOIC127P600X175-8N, symbol EPCS1SI8N:EPCS1SI8N
- added U4: AMS1117-3.3, Package_TO_SOT_SMD:SOT-223-3_TabPin2, symbol Regulator_Linear:AMS1117-3.3
- added U5: AMS1117-1.5, Package_TO_SOT_SMD:SOT-223-3_TabPin2, symbol Regulator_Linear:AMS1117-1.5
- C12: footprint Capacitor_SMD:CP_Elec_5x5.9 -> Capacitor_THT:CP_Radial_D5.0mm_P2.50mm
Connections:
- net +5V: now also C13.1, C15.1, U4.3 (VI), U5.3 (VI); no longer C10.1, C2.1, C3.1, C4.1, C5.1, C6.2, C7.1, C8.1, C9.2, U1.18 (VCCIO1), U1.31 (VCCIO4), U1.33 (VCCINT), U1.44 (VCCINT), U1.46 (VCCIO4), U1.59 (VCCIO3), U1.80 (VCCIO2), U1.82 (VCCINT), U1.9 (VCCA_PLL1), U1.93 (VCCINT), U1.95 (VCCIO2)
- net GND: now also U1.14 (MSEL0), U1.15 (MSEL1), U1.62 (TCK), C11.2, C13.2, C14.2, C15.2, C16.2, C17.1, J1.10 (Pin_10), J1.2 (Pin_2), U3.4 (GND), U4.1 (GND), U5.1 (GND)
- net C_CE: now reaches U1.13 (NCE)
- net C_CE: now also J1.6 (Pin_6), RN9.5 (R4.2)
- net AS_CK: now reaches U1.16 (DCLK)
- net AS_CK: now also U3.6 (DCLK)
- net C_DONE: now reaches U1.60 (CONF_DONE)
- net C_DONE: now also J1.3 (Pin_3), RN9.8 (R1.2)
- net C_STAT: now reaches U1.61 (NSTATUS)
- net C_STAT: now also RN9.6 (R3.2)
- net +3.3V: now reaches U1.63 (TMS)
- net +3.3V: now also C10.1, C2.1, C3.1, C4.1, C5.1, U1.18 (VCCIO1), U1.31 (VCCIO4), U1.46 (VCCIO4), U1.59 (VCCIO3), U1.67 (TDI), U1.80 (VCCIO2), U1.95 (VCCIO2), C11.1, C14.1, J1.4 (Pin_4), RN9.1 (R1.1), RN9.2 (R2.1), RN9.3 (R3.1), RN9.4 (R4.1), U3.3 (VCC_2), U3.7 (VCC_3), U3.8 (VCC), U4.2 (VO)
- net AS_DI: now reaches U1.7 (DATA0)
- net AS_DI: now also J1.7 (Pin_7), U3.2 (DATA)
- net C_CONF: now reaches U1.8 (NCONFIG)
- net C_CONF: now also J1.5 (Pin_5), RN9.7 (R2.2)
- new net: C17.2, R1.2, U1.9 (VCCA_PLL1)
- new net +1V5: C16.1, C6.2, C7.1, C8.1, C9.2, R1.1, U1.33 (VCCINT), U1.44 (VCCINT), U1.82 (VCCINT), U1.93 (VCCINT), U5.2 (VO)
- new net AS_CS: U3.1 (NCS)
- new net AS_DO: J1.9 (Pin_9), U3.5 (ASDI)
- no-connect marks 11 -> 13
Other:
- moved on the sheet: C1, C2, C3, C4, C5, C6, C7, C8, C9, U1A

Commit message: wip
Parts:
- added J1: Conn_01x03_Pin, symbol Connector:Conn_01x03_Pin
- added J3: JTAG_DEBUG, Connector_PinHeader_2.54mm:PinHeader_2x05_P2.54mm_Vertical, symbol Connector_Generic:Conn_02x05_Odd_Even
- added JP1, JP2, JP3: Jumper_2_Open, symbol Jumper:Jumper_2_Open
- added R1: 10K, symbol Device:R
- added R2, R3, R4: 1K, symbol Device:R
- added U6: ESP-01, Connector_PinSocket_2.54mm:PinSocket_2x04_P2.54mm_Vertical, symbol ESP8266:ESP-01v090
- C17: value 0.1uF -> 100nF
- J2: renamed from J1; value Conn_02x05_Odd_Even -> AS
- renumbered C2 to C1, C6 to C10, C15 to C11, C7 to C12, C8 to C13, C9 to C14, C16 to C15, C11 to C16, C12 to C2, C1 to C4, C13 to C5, C4 to C6, C5 to C7, C14 to C8, C10 to C9, R1 to R5, RN9 to RN1, RN1 to RN2, RN2 to RN3, RN3 to RN4, RN4 to RN5, RN5 to RN6, RN8 to RN7, RN7 to RN8, RN6 to RN9, U4 to U1, U5 to U3, U1 to U4, U3 to U5
Connections:
- net +3.3V: now also R2.1, R3.1, U6.7 (VCC); no longer U4.63 (TMS), U4.67 (TDI)
- net +5V: now also R1.2
- net A14: now also U2.5 (A14)
- net AS_CK: now also J2.1 (Pin_1)
- net GND: now also U2.10 (A16), J1.1 (Pin_1), J3.10 (Pin_10), J3.2 (Pin_2), R4.1, U6.2 (GND); no longer U4.62 (TCK)
- net MA14: no longer U2.5 (A14)
- net MA15: no longer U2.11 (A15)
- net MA16: no longer U2.10 (A16)
- net RD: no longer U2.32 (OE#)
- net JT_TDO: now reaches U4.64 (TDO)
- net JT_TDO: now also J3.3 (Pin_3)
- net CS1: now reaches BUS1.1 (~{CS1})
- net CS1: now also JP1.2 (B)
- net CS2: now reaches BUS1.2 (~{CS2})
- net CS2: now also JP2.2 (B)
- net CS12: now reaches BUS1.3 (~{CS12})
- net CS12: now also JP3.2 (B)
- net WAIT: now reaches BUS1.7 (~{WAIT})
- net WAIT: now also RN7.7 (R2.2)
- net at U4.72 (IO): now also RN7.2 (R2.1)
- new net: JP1.1 (A), JP2.1 (A), JP3.1 (A), U2.32 (OE#)
- new net: J1.3 (Pin_3), R1.1
- new net A15_SW: J1.2 (Pin_2), U2.11 (A15)
- new net JT_TCK: J3.1 (Pin_1), R4.2, U4.62 (TCK)
- new net JT_TDI: J3.9 (Pin_9), R3.2, U4.67 (TDI)
- new net JT_TMS: J3.5 (Pin_5), R2.2, U4.63 (TMS)
- no-connect marks 13 -> 11
Other:
- moved on the sheet: BUS1, C1, C10, C11, C12, C13, C14, C15, C16, C17, C2, C3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

Commit message: wip
Parts:
- removed J1: Conn_01x03_Pin, symbol Connector:Conn_01x03_Pin
- removed JP1, JP2, JP3: Jumper_2_Open, symbol Jumper:Jumper_2_Open
- removed R1: 10K, symbol Device:R
- removed U2: AM29F010B, Package_SO:TSOP-I-32_18.4x8mm_P0.5mm, symbol AM29F010B:AM29F010B
- removed U4: EP1C3T100C8N, libraries:QFP50P1600X1600X120-100N, symbol EP1C3T100C8N:EP1C3T100C8N
- removed U6: ESP-01, Connector_PinSocket_2.54mm:PinSocket_2x04_P2.54mm_Vertical, symbol ESP8266:ESP-01v090
- added Cart1: MSX-cartridge_dummy, libraries:LOGO_MSX, symbol CRISAG:MSX-cartridge_dummy
- added J3: Conn_01x02, Connector_PinHeader_2.54mm:PinHeader_1x02_P2.54mm_Vertical, symbol Connector_Generic:Conn_01x02
- added RN1, RN10: 330, Resistor_SMD:R_Array_Convex_4x0603, symbol Device:R_Pack04_Split
- added U2: ~, Package_SO:TSOP-I-32_18.4x8mm_P0.5mm, symbol AM29LV010B:AM29LV010B
- added U5: EP1C3T144C8N, libraries:QFP50P2200X2200X160-144N, symbol EP1C3T144C8N:EP1C3T144C8N
- added U6: ESP-01, libraries:MODULE_ESP-01, symbol ESP-01:ESP-01
- C1, C10, C12, C13, C14, C16, C3, C4, C6, C7, C9: footprint Capacitor_SMD:C_0805_2012Metric_Pad1.18x1.45mm_HandSolder -> Capacitor_SMD:C_0603_1608Metric
- C11, C15, C17, C5, C8: footprint Capacitor_SMD:C_0805_2012Metric -> Capacitor_SMD:C_0603_1608Metric
- J1: renamed from J2; footprint Connector_PinHeader_2.54mm:PinHeader_2x05_P2.54mm_Vertical -> Connector_IDC:IDC-Header_2x05_P2.54mm_Vertical
- J2: renamed from J3; footprint Connector_PinHeader_2.54mm:PinHeader_2x05_P2.54mm_Vertical -> Connector_IDC:IDC-Header_2x05_P2.54mm_Vertical
- R1: renamed from R5; footprint Resistor_SMD:R_0805_2012Metric -> Resistor_SMD:R_0603_1608Metric
- R2, R3, R4: footprint (none) -> Resistor_SMD:R_0603_1608Metric
- renumbered RN1 to RN11, U5 to U4
Connections:
- net CS2 is gone; now on an unnamed net: BUS1.2 (~{CS2})
- net SLTSL is gone; now on an unnamed net: BUS1.4 (~{SLTSL})
- net +1V5: now also U5.117 (VCCINT), U5.135 (VCCINT_2), U5.46 (VCCINT_2), U5.64 (VCCINT); no longer R1.1
- net +3.3V: now also C4.2, R1.2, U2.8 (VCC), U5.102 (VCCIO3), U5.115 (VCCIO2_2), U5.137 (VCCIO2), U5.29 (VCCIO1), U5.44 (VCCIO4_2), U5.66 (VCCIO4), U5.8 (VCCIO1_2), U5.81 (VCCIO3_2), U6.5 (VCC)
- net +5V: now also J3.2 (Pin_2); no longer C4.2
- net AS_CK: now also U5.24 (DCLK)
- net AS_CS: now also U5.74 (IO_3)
- net AS_DI: now also U5.13 (DATA0)
- net AS_DO: now also U5.73 (IO_2)
- net C_CE: now also U5.21 (NCE)
- net C_CONF: now also U5.14 (NCONFIG)
- net C_DONE: now also U5.86 (CONF_DONE)
- net C_STAT: now also U5.87 (NSTATUS)
- net GND: now also J3.1 (Pin_1), U2.24 (VSS), U5.101 (GND_4), U5.116 (GND_3), U5.118 (GND_5), U5.136 (GND_6), U5.138 (GND), U5.18 (GNDA_PLL1), U5.19 (GNDG_PLL1), U5.22 (MSEL0), U5.23 (MSEL1), U5.30 (GND_2), U5.43 (GND_4), U5.45 (GND_5), U5.63 (GND), U5.65 (GND_6), U5.80 (GND_2), U5.9 (GND_3), U6.1 (GND)
- net JT_TCK: now also U5.88 (TCK)
- net JT_TDI: now also U5.95 (TDI)
- net JT_TDO: now also U5.90 (TDO)
- net JT_TMS: now also U5.89 (TMS)
- net at RN6.5 (R4.2): now also BUS1.8 (~{INT})
- net SLT_A5: now reaches RN4.5 (R4.2)
- net SLT_A5: now also U5.107 (IO_24)
- net at RN8.6 (R3.2): now also BUS1.22 (A6)
- net at BUS1.12 (~{MERQ}): now also RN7.7 (R2.2)
- net at BUS1.6 (~{RFSH}): now also RN6.6 (R3.2)
- net at BUS1.9 (~{M1}): now also RN2.1 (R1.1)
- net at C17.2: now also R1.1, U5.15 (VCCA_PLL1); no longer R1.2
- net SLT_M1: now reaches RN2.8 (R1.2)
- net SLT_M1: now also U5.132 (IO_45)
- net SLT_IORQ: now reaches RN2.7 (R2.2)
- net SLT_IORQ: now also U5.130 (IO_43)
- net SLT_WR: now reaches RN2.6 (R3.2)
- net SLT_WR: now also U5.128 (IO_41)
- net SLT_RESET: now reaches RN2.5 (R4.2)
- net SLT_RESET: now also U5.126 (IO_39)
- net at RN3.1 (R1.1): now also BUS1.17 (A9)
- net at RN3.2 (R2.1): now also BUS1.19 (A11)
- net at RN3.3 (R3.1): now also BUS1.21 (A7)
- net at RN3.4 (R4.1): now also BUS1.23 (A12)
- net SLT_A14: now reaches RN4.8 (R1.2)
- net SLT_A14: now also U5.113 (IO_30)
- net SLT_A1: now reaches RN4.7 (R2.2)
- net SLT_A1: now also U5.111 (IO_28)
- net SLT_A3: now reaches RN4.6 (R3.2)
- net SLT_A3: now also U5.109 (IO_26)
- net at RN5.1 (R1.1): now also BUS1.33 (D1)
- net at RN5.2 (R2.1): now also BUS1.35 (D3)
- net at RN5.3 (R3.1): now also BUS1.37 (D5)
- net at RN5.4 (R4.1): now also BUS1.39 (D7)
- net SLT_A13: now reaches RN9.1 (R1.1)
- net SLT_A13: now also U5.112 (IO_29)
- net SLT_A0: now reaches RN9.2 (R2.1)
- net SLT_A0: now also U5.110 (IO_27)
- net SLT_A2: now reaches RN9.3 (R3.1)
- net SLT_A2: now also U5.108 (IO_25)
- net SLT_A4: now reaches RN9.4 (R4.1)
- net SLT_A4: now also U5.106 (IO_23)
- net at RN8.8 (R1.2): now also BUS1.18 (A15)
- net at RN8.7 (R2.2): now also BUS1.20 (A10)
- net at RN8.5 (R4.2): now also BUS1.24 (A8)
- net SLT_BUSDIR: now reaches RN7.1 (R1.1)
- net SLT_BUSDIR: now also U5.131 (IO_44)
- net SLT_MERQ: now reaches RN7.2 (R2.1)
- net SLT_MERQ: now also U5.129 (IO_42)
- net SLT_RD: now reaches RN7.3 (R3.1)
- net SLT_RD: now also U5.127 (IO_40)
- net at RN7.6 (R3.2): now also BUS1.14 (~{RD})
- net A0: no longer names the net of BUS1.28 (A0)
- net A0: now also RN9.7 (R2.2); no longer RN5.8 (R1.2)
- net A1: no longer names the net of BUS1.27 (A1)
- net A1: now also RN4.2 (R2.1); no longer RN5.7 (R2.2)
- net A10: no longer names the net of RN9.8 (R1.2)
- net A10: now also BUS1.26 (A13); no longer BUS1.20 (A10)
- removed net A11: BUS1.19 (A11), RN9.7 (R2.2)
- net A12 renamed SLT_SLTSL
- net SLT_SLTSL: now also U5.140 (IO_49); no longer BUS1.23 (A12)
- net A13 renamed SLT_D5
- net SLT_D5: now also U5.99 (IO_18); no longer BUS1.26 (A13)
- net A14: no longer names the net of BUS1.25 (A14)
- net A14: now also RN4.1 (R1.1); no longer RN5.5 (R4.2)
- net A15: no longer names the net of RN9.6 (R3.2)
- net A15: now also BUS1.30 (A2); no longer BUS1.18 (A15)
- net A2: no longer names the net of RN4.3 (R3.1)
- net A2: now also BUS1.29 (A3); no longer BUS1.30 (A2)
- net A3: no longer names the net of RN4.4 (R4.1)
- net A3: now also BUS1.31 (A5); no longer BUS1.29 (A3)
- net A4: no longer names the net of BUS1.32 (A4)
- net A4: now also RN9.5 (R4.2); no longer RN4.1 (R1.1)
- removed net A5: BUS1.31 (A5), RN4.2 (R2.1)
- net A6 renamed SLT_RFSH
- net SLT_RFSH: now also U5.139 (IO_48); no longer BUS1.22 (A6)
- net A7 renamed SLT_INT
- net SLT_INT: now also U5.133 (IO_46); no longer BUS1.21 (A7)
- net A8 renamed SLT_CS2
- net SLT_CS2: now also U5.142 (IO_51); no longer BUS1.24 (A8)
- removed net A9: BUS1.17 (A9), RN9.5 (R4.2)
- net BUSDIR: no longer names the net of BUS1.10 (~{BUSDIR})
- net BUSDIR: now also RN7.8 (R1.2); no longer RN8.4 (R4.1)
- net CS1: no longer names the net of BUS1.1 (~{CS1})
- net CS1: now also RN1.1 (R1.1)
- net CS12: no longer names the net of BUS1.3 (~{CS12})
- net CS12: now also RN1.2 (R2.1)
- net D0: no longer names the net of BUS1.34 (D0)
- net D0: now also RN10.8 (R1.2); no longer RN3.6 (R3.2)
- net D1 renamed SLT_A12
- net SLT_A12: now also U5.119 (IO_32); no longer BUS1.33 (D1)
- net D2: no longer names the net of BUS1.36 (D2~{})
- net D2: now also RN10.7 (R2.2); no longer RN3.8 (R1.2)
- net D3 renamed SLT_A11
- net SLT_A11: now also U5.123 (IO_36); no longer BUS1.35 (D3)
- net D4: no longer names the net of RN2.3 (R3.1)
- net D4: now also BUS1.13 (~{WR}); no longer BUS1.38 (D4)
- net D5: no longer names the net of RN2.4 (R4.1)
- net D5: now also BUS1.15 (~{RESET}); no longer BUS1.37 (D5)
- net D6: no longer names the net of BUS1.40 (D6)
- net D6: now also RN10.5 (R4.2); no longer RN2.1 (R1.1)
- net D7: no longer names the net of RN2.2 (R2.1)
- net D7: now also BUS1.11 (~{IORQ}); no longer BUS1.39 (D7)
- net IORQ renamed SLT_A6
- net SLT_A6: now also U5.120 (IO_33); no longer BUS1.11 (~{IORQ})
- net RD renamed SLT_A15
- net SLT_A15: now also U5.124 (IO_37); no longer BUS1.14 (~{RD})
- removed net RESET: BUS1.15 (~{RESET}), RN7.8 (R1.2)
- net WAIT: no longer names the net of BUS1.7 (~{WAIT})
- net WAIT: now also RN1.4 (R4.1); no longer RN7.7 (R2.2)
- net WR renamed SLT_A10
- net SLT_A10: now also U5.122 (IO_35); no longer BUS1.13 (~{WR})
- new net: BUS1.38 (D4), RN10.6 (R3.2)
- new net ESP_CHPD: U5.70 (IO_47), U6.7 (CH_PD)
- new net ESP_RST: U5.69 (IO_46), U6.6 (~{RST})
- new net ESP_RXD: U5.68 (IO_45), U6.4 (RXD)
- new net ESP_TXD: U5.71 (IO_48), U6.8 (TXD)
- new net ROM_A0: U2.20 (A0), U5.41 (IO_26)
- new net ROM_A1: U2.19 (A1), U5.42 (IO_27)
- new net ROM_A10: U2.31 (A10), U5.35 (IO_20)
- new net ROM_A11: U2.1 (A11), U5.1 (IO_2)
- new net ROM_A12: U2.12 (A12), U5.11 (IO_10)
- new net ROM_A13: U2.4 (A13), U5.4 (IO_5)
- new net ROM_A14: U2.5 (A14), U5.5 (IO_6)
- new net ROM_A15: U2.11 (A15), U5.10 (IO_9)
- new net ROM_A16: U2.10 (A16), U5.7 (IO_8)
- new net ROM_A2: U2.18 (A2), U5.47 (IO_28)
- new net ROM_A3: U2.17 (A3), U5.48 (IO_29)
- new net ROM_A4: U2.16 (A4), U5.27 (IO_14)
- new net ROM_A5: U2.15 (A5), U5.26 (IO_13)
- new net ROM_A6: U2.14 (A6), U5.25 (IO_12)
- new net ROM_A7: U2.13 (A7), U5.12 (IO_11)
- new net ROM_A8: U2.3 (A8), U5.3 (IO_4)
- new net ROM_A9: U2.2 (A9), U5.2 (IO_3)
- new net ROM_CE: U2.30 (CE#), U5.34 (IO_19)
- new net ROM_D0: U2.21 (DQ0), U5.40 (IO_25)
- new net ROM_D1: U2.22 (DQ1), U5.39 (IO_24)
- new net ROM_D2: U2.23 (DQ2), U5.38 (IO_23)
- new net ROM_D3: U2.25 (DQ3), U5.37 (IO_22)
- new net ROM_D4: U2.26 (DQ4), U5.28 (IO_15)
- new net ROM_D5: U2.27 (DQ5), U5.31 (IO_16)
- new net ROM_D6: U2.28 (DQ6), U5.32 (IO_17)
- new net ROM_D7: U2.29 (DQ7), U5.33 (IO_18)
- new net ROM_OE: U2.32 (OE#), U5.36 (IO_21)
- new net ROM_WR: U2.7 (WE#), U5.6 (IO_7)
- new net SLT_A7: RN3.6 (R3.2), U5.121 (IO_34)
- new net SLT_A8: RN8.4 (R4.1), U5.114 (IO_31)
- new net SLT_A9: RN3.8 (R1.2), U5.125 (IO_38)
- new net SLT_CS1: RN1.8 (R1.2), U5.143 (IO_52)
- new net SLT_CS12: RN1.7 (R2.2), U5.141 (IO_50)
- new net SLT_D0: RN10.1 (R1.1), U5.104 (IO_21)
- new net SLT_D1: RN5.8 (R1.2), U5.105 (IO_22)
- new net SLT_D2: RN10.2 (R2.1), U5.100 (IO_19)
- new net SLT_D3: RN5.7 (R2.2), U5.103 (IO_20)
- new net SLT_D4: RN10.3 (R3.1), U5.98 (IO_17)
- new net SLT_D6: RN10.4 (R4.1), U5.96 (IO_15)
- new net SLT_D7: RN5.5 (R4.2), U5.97 (IO_16)
- new net SLT_WAIT: RN1.5 (R4.2), U5.134 (IO_47)
- no-connect marks 11 -> 41
Other:
- moved on the sheet: C17, C4, R1

Commit message: routing
Parts:
- added C16: 100nF, Capacitor_SMD:C_0603_1608Metric, symbol Device:C
- added LogoTRH1: LogoTRH, libraries:TRH, symbol CRISAG:MSX-cartridge_dummy
- added R1: 330, Resistor_SMD:R_0603_1608Metric, symbol Device:R
- added Y1: SG-310SCN_50.0000MJ3, libraries:SG310SCN500000MJ3, symbol SG-310SCN_50_0000MJ3:SG-310SCN_50.0000MJ3
- LogoMSX1: renamed from Cart1; value MSX-cartridge_dummy -> LogoMSX
- renumbered C16 to C18, J3 to J1, J1 to J2, J2 to J3, R1 to R2, R2 to R3, R3 to R4, R4 to R5
Connections:
- net +3.3V: now also J3.4 (Pin_4), C16.1, Y1.4 (VCC)
- net GND: now also U5.17 (CLK1), C16.2, Y1.2 (GND)
- net SLT_CLK: now reaches U5.93 (CLK2)
- net SLT_CLK: now also R1.2
- net at BUS1.42 (CLOCK): now also R1.1
- net at U5.16 (CLK0): now also Y1.3 (OUT)
- no-connect marks 41 -> 44
Other:
- moved on the sheet: C1, C10, C11, C15, C17, C18, C5, C7, C8, C9, J2, J3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

Commit message: First tests with the verilog code
Parts:
- U2: value ~ -> AM29LV010B
Changed lines of the file:
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@@
 		(on_board yes)
 		(dnp no)
-		(fields_autoplaced yes)
 		(property "Reference" "U2"
 			(at 166.9289 190.5 0)
@@
 			)
 		)
-		(property "Value" "~"
-			(at 161.29 209.55 0)
+		(property "Value" "AM29LV010B"
+			(at 172.974 188.214 0)
 			(effects
 				(font
